File: pcb/af4-trigger-hat-backups/af4-trigger-hat-pre-LED-resistor-change.kicad_pcb (KiCad board)
At the start: 2 copper layers, 57 x 50 mm, 28 parts, among them J1 PJ-079BH, J2 SJ1-3523N, J3 EXT1, J4 EXT2, U1 AQY212GS, U2 LM1117MPX-ADJ

Commit message: pcb: fix three non-existent MPNs, split LED series resistors
Three part numbers in the rev D BOM did not exist. All were
well-formed under their manufacturer's naming scheme but return no
stocked part; PCBWay's sourcing flagged one and silently substituted
the other two.

  F1  1206L010/60YR      -> 1206L010/60WR
      The 1206L suffix is a reel-quantity code (WR=3000, YR=4000);
      the 60 V value ships only as /60WR. Trip current is 0.25 A,
      not the 0.30 A the docs claimed.
  C1  GRM31CR71H106KA12L -> GRM31CR61H106KA12L
      R7=X7R, R6=X5R. Murata makes no 10 uF 50 V X7R in 1206; that
      C/V needs a 1210. X5R is correct for input bulk.
  D5  APT2012SYC         -> APT2012SYCK
      No APT2012SYC exists. SYCK is 590 nm, 150 mcd at 20 mA.

Separately, D3 was under-driven ~10x. R6/R7 shared a 10 k value, but
APT2012SGC is 12 mcd typ / 5 mcd min at 20 mA against APT2012SYCK's
150 mcd -- roughly 12x apart in efficiency. At 0.82 mA the green sat
near 0.5 mcd, invisible through the lid's 3.5 mm sight hole. Split
the line: R6 = 1.0 k (8.2 mA), R7 = 6.8 k (1.2 mA). R2 stays 10 k.
BOM goes 18 -> 20 lines; placements unchanged at 21.

No gerber change: resistor values live on hidden F.Fab text, so the
fab package PCBWay already holds remains valid.

The other 15 MPNs were verified against live distributor listings
and are correct, as are the LM1117 minimum-load, output-cap ESR and
R1 drive-current calculations (re-derived from datasheets).
Parts:
- R6: value 1k0 -> 10k
- R7: value 6k8 -> 10k
Changed lines of the file:
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@@
         (effects (font (size 1 1) (thickness 0.15)))
     )
-    (fp_text value "6k8" (at 0 1.65) (layer "F.Fab") hide
+    (fp_text value "10k" (at 0 1.65) (layer "F.Fab") hide
         (effects (font (size 1 1) (thickness 0.15)))
     )
@@
         (effects (font (size 1 1) (thickness 0.15)))
     )
-    (fp_text value "1k0" (at 0 1.65) (layer "F.Fab") hide
-        (effects (font (size 1 1) (thickness 0.15)))
-    )
+    (fp_text value "10k" (at 0 1.65) (layer "F.Fab") hide
+        (effects (font (size 1 1) (thickness 0.15)))
+    )
