File: pcb/af4-trigger-hat.kicad_pcb (KiCad board)
At the start: 2 copper layers, 57 x 50 mm, 28 parts, among them J1 PJ-079BH, J2 SJ1-3523N, J3 EXT1, J4 EXT2, U1 AQY212GS, U2 LM1117MPX-ADJ

Commit message: pcb: rebuild U1 land pattern from Panasonic's drawing
U1 was on SO-4_4.4x2.3mm_P1.27mm, a 1.27 mm-pitch generic SO-4 whose
library description points at an OPTEK OPIA403. The AQY212GS is a
Panasonic GU SOP4 at 2.54 mm pitch, so every pin missed its pad by
0.635 mm. The board could not be built and the Gerbers sent to PCBWay
were invalid.

U1 now uses a project-local footprint authored from the "Recommended
mounting pad" drawing in semi_eng_gu_sop4_1a.pdf:

  pcb/footprints/aF4.pretty/AQY212GS_SOP4_Panasonic.kicad_mod
  pad 0.8 mm across pitch x 1.2 mm along the lead axis
  centres 2.54 mm on pitch, 6.00 mm across the span

gen_pcb.py's load() now prefers a project-local footprints/ directory
over the stock KiCad libraries.

An interim fix used KiCad's SO-4_4.4x4.3mm_P2.54mm, which matches on
pitch, body and pad centres but has its pads rotated 90 degrees --
0.8 mm along the lead axis where Panasonic asks for 1.2. It would have
mounted with no toe fillet. Matching dimensions beats matching a name
and is still not the same as reading the recommended-pad drawing.

Also from the independent audit:
  - D2 said SMAJ15A in gen_pcb.py while the BOM said SMAJ13A
  - "44 THT joints" was fiction; the real count is 28, now computed
    from the board's PTH pads. PCBWay prices hand-soldered joints
  - circuit diagram showed D2 upstream of D1; the board wires it
    downstream
  - LM1117 dropout does not collapse at light load; it is a quasi-LDO
    with a nearly flat ~1 V dropout
  - R5 runs at ~96 mW against an 0805's 125 mW rating
  - AQY212 turn-off current is 0.3 mA min, so GPIO13's 0.72-0.85 mA of
    boot leakage was over 2x the guaranteed-off threshold. The move to
    GPIO32 was mandatory, not insurance

Verification: DRC 61 items, identical in class and count to a baseline
regenerated with the old footprint. 0 clearance, 0 courtyard, 0 hole,
0 copper-to-edge, 0 unconnected, 0 mask bridges. No plated slot under
0.70 mm. BOM == PARTS == board refs. True logic-to-power cre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
Parts:
- D2: value SMAJ15A -> SMAJ13A
- U1: footprint SO-4_4.4x2.3mm_P1.27mm -> AQY212GS_SOP4_Panasonic
Routing:
- net LED_A: track 5.30 -> 4.52 mm

Commit message: pcb: relabel rev D -> rev E; board proven geometrically identical
Other:
- board text added: "rev E inD aF4 frozen feeder"
- board text removed: "rev D inD aF4 frozen feeder"
